Commit message: Update BlueRov2.urdf.xacro
change buoyancy setting

File: model/BlueRov2.urdf.xacro (robot description, xacro)
@@ -102,4 +102,10 @@
     </collision-->
     <buoyancy>
+        <compensation>1.01</compensation>
+        <origin xyz= "0.0 0.0 -0.0"/>
+        <limit radius=".5"/>
+        <damping xyz="60 100 100" rpy="20 50 50"/>
+    </buoyancy>
+    <!--buoyancy>
         <compensation>0.2525</compensation>
         <origin xyz= "0.12585 0.111 -0.8945"/>
@@ -116,5 +122,5 @@
         <compensation>0.2525</compensation>
         <origin xyz= "0.12585 -0.111 -0.8945"/>
-    </buoyancy>
+    </buoyancy-->
   </link>
   <link name="camera_link">
