Commit message: add obstacle model file

File: urdfs/BlueRov2.xacro (robot description, xacro)
@@ -4,4 +4,5 @@
   <!--<xacro:property name="buoy" value="0.2525" />-->
   <xacro:property name="buoy" value="0.1263" />
+  <xacro:property name="PI" value="3.1415926" />
   <link name='base_link'>
     <inertial>

Commit message: Add an upward camera to the URDF filse of the UUV

File: urdfs/BlueRov2.xacro (robot description, xacro)
@@ -349,5 +349,5 @@
     </joint>
     <!--<allow_auto_disable>1</allow_auto_disable>-->
-    <link name="camera_link">
+    <!--link name="camera_link">
       <visual>
         <origin xyz="0 0 0" rpy="0 0 0" />
@@ -416,5 +416,77 @@
     <origin xyz= "0.2 0.0 0.2" rpy="0 0 0" />
     <axis xyz="0 0 1" />
-  </joint>
+  </joint-->
+  <link name="camera_visual_link">
+    <visual>
+      <geometry>
+        <cylinder length="0.3" radius="0.05"/>
+      </geometry>
+      <material name="white">
+        <color rgba="1 1 1 1"/>
+      </material>
+    </visual>
+  </link>
+  <joint name="camera_visual_joint" type="fixed">
+    <parent link="base_link"/>
+    <child link="camera_visual_link"/>
+    <origin rpy="${PI/2.0} ${-PI/2.0} 0" xyz="0 0.0 0.2"/>
+    <axis xyz="1 0 0" />
+  </joint>
+  <link name="camera_link">
+    <!--visual>
+      <geometry>
+        <cylinder length="0.3" radius="0.05"/>
+      </geometry>
+      <material name="white">
+        <color rgba="1 1 1 1"/>
+      </material>
+    </visual-->
+  </link>
+  <joint name="camera_joint" type="fixed">
+    <parent link="base_link"/>
+    <child link="camera_link"/>
+    <origin rpy="${PI/2.0} ${-PI/2.0} ${PI/2.0}" xyz="0 0.0 0.2"/>
+    <axis xyz="1 0 0" />
+  </joint>
+  <!-- camera -->
+  <gazebo reference="camera_link">
+    <sensor type="camera" name="camera1">
+      <always_on>true</always_on>
+      <visualize>false</visualize>
+      <update_rate>10.0</update_rate>
+      <camera name="head">
+        <horizontal_fov>2.09</horizontal_fov>
+        <image>
+          <width>1920</width>
+          <height>1080</height>
+          <format>R8G8B8</format>
+        </image>
+        <clip>
+          <near>0.01</near>
+          <far>500</far>
+        </clip>
+        <noise>
+          <type>gaussian</type>
+          <mean>0.0</mean>
+          <stddev>0.007</stddev>
+        </noise>
+      </camera>
+      <plugin name="camera_controller" filename="libgazebo_ros_camera.so">
+        <alwaysOn>true</alwaysOn>
+        <visualize>false</visualize>
+        <updateRate>30.0</updateRate>
+        <cameraName>camera</cameraName>
+        <imageTopicName>image_raw</imageTopicName>
+        <cameraInfoTopicName>camera_info</cameraInfoTopicName>
+        <frameName>camera_link</frameName>
+        <hackBaseline>0.07</hackBaseline>
+        <distortionK1>0.0</distortionK1>
+        <distortionK2>0.0</distortionK2>
+        <distortionK3>0.0</distortionK3>
+        <distortionT1>0.0</distortionT1>
+        <distortionT2>0.0</distortionT2>
+      </plugin>
+    </sensor>
+  </gazebo>
   <gazebo>
     <plugin name="ArduPilotPlugin" filename="libArduPilotPlugin.so">

Commit message: Added an upward camera to the UUV urdf model.

File: urdfs/BlueRov2.xacro (robot description, xacro)
@@ -2,6 +2,5 @@
 <robot name="BlueRov2" xmlns:xacro="http://ros.org/wiki/xacro">
   <!-- properties -->
-  <!--<xacro:property name="buoy" value="0.2525" />-->
-  <xacro:property name="buoy" value="0.1263" />
+  <xacro:property name="buoy" value="0.2525" />
   <xacro:property name="PI" value="3.1415926" />
   <link name='base_link'>
@@ -480,4 +479,64 @@
         <cameraInfoTopicName>camera_info</cameraInfoTopicName>
         <frameName>camera_link</frameName>
+        <hackBaseline>0.07</hackBaseline>
+        <distortionK1>0.0</distortionK1>
+        <distortionK2>0.0</distortionK2>
+        <distortionK3>0.0</distortionK3>
+        <distortionT1>0.0</distortionT1>
+        <distortionT2>0.0</distortionT2>
+      </plugin>
+    </sensor>
+  </gazebo>
+  <link name="front_camera_visual_link">
+    <visual>
+      <geometry>
+        <cylinder length="0.02" radius="0.02"/>
+      </geometry>
+      <material name="white">
+        <color rgba="1 1 1 1"/>
+      </material>
+    </visual>
+  </link>
+  <joint name="front_camera_visual_joint" type="fixed">
+    <parent link="base_link"/>
+    <child link="front_camera_visual_link"/>
+    <origin rpy="0 1.57 0" xyz="0.2 0 0.3"/>
+    <axis xyz="1 0 0" />
+  </joint>
+  <link name="front_camera_link">
+  </link>
+  <joint name="front_camera_joint" type="fixed">
+    <parent link="base_link"/>
+    <child link="front_camera_link"/>
+    <origin rpy="0 0 0" xyz="0.2 0.0 0.3"/>
+    <axis xyz="1 0 0" />
+  </joint>
+  <gazebo reference="front_camera_link">
+    <sensor type="camera" name="front_camera">
+      <update_rate>30.0</update_rate>
+      <camera name="front_camera">
+        <horizontal_fov>1.3962634</horizontal_fov>
+        <image>
+          <width>1280</width>
+          <height>720</height>
+          <format>R8G8B8</format>
+        </image>
+        <clip>
+          <near>0.02</near>
+          <far>300</far>
+        </clip>
+        <noise>
+          <type>gaussian</type>  <!-- Noise is sampled independently per pixel on each frame. That pixel's noise value is added to each of its color channels, which at that point lie in the range [0,1]. -->
+	  <mean>0.0</mean>
+          <stddev>0.007</stddev>
+        </noise>
+      </camera>
+      <plugin name="front_camera_controller" filename="libgazebo_ros_camera.so">
+        <alwaysOn>true</alwaysOn>
+        <updateRate>0.0</updateRate>
+        <cameraName>uuv_front</cameraName>
+	<imageTopicName>image</imageTopicName>
+        <cameraInfoTopicName>camera_info</cameraInfoTopicName>
+	<frameName>BlueRov2/front_camera_link</frameName>
         <hackBaseline>0.07</hackBaseline>
         <distortionK1>0.0</distortionK1>
@@ -591,4 +650,5 @@
       <surface>0 0 0</surface>
       <updateRate>.001</updateRate>
+      <wave_model>ocean_waves</wave_model>
       <link name="base_link">
         <buoyancy>

Commit message: edit size of the collection mechanism

File: urdfs/BlueRov2.xacro (robot description, xacro)
@@ -121,5 +121,5 @@
     <child link="collector_left" />
     <parent link="base_link" />
-    <origin xyz="0 0.15 0.23" rpy="0 0 0" />
+    <origin xyz="0 0.175 0.23" rpy="0 0 0" />
     <axis xyz="0 0 1" />
   </joint>
@@ -154,5 +154,5 @@
     <child link="collector_right" />
     <parent link="base_link" />
-    <origin xyz="0 -0.15 0.23" rpy="0 0 0" />
+    <origin xyz="0 -0.175 0.23" rpy="0 0 0" />
     <axis xyz="0 0 1" />
   </joint>
@@ -163,5 +163,5 @@
     <visual>
       <geometry>
-        <box size="0.01 0.30 0.15" />
+        <box size="0.01 0.35 0.15" />
       </geometry>
       <material name="black"/>
@@ -196,5 +196,5 @@
     <visual>
       <geometry>
-        <box size="0.01 0.30 0.15" />
+        <box size="0.01 0.35 0.15" />
       </geometry>
       <material name="black"/>
